File: connectors.kicad_sch (KiCad schematic)
At the start: 4 parts, among them J1 Conn_01x04_Pin, J2 Conn_01x04_Pin, J3 Conn_01x09_Pin, J4 Conn_02x03_Odd_Even

Commit message: finished wiring connector sheet
Connections:
- net D2: now reaches J3.1 (Pin_1)
- net D3: now reaches J3.2 (Pin_2)
- net D4: now reaches J3.3 (Pin_3)
- net D5: now reaches J3.4 (Pin_4)
- net D6: now reaches J3.5 (Pin_5)
- net D7: now reaches J3.6 (Pin_6)
- net D8: now reaches J3.7 (Pin_7)
- net GND: now reaches J3.8 (Pin_8)
- net GND: now also J1.1 (Pin_1), J2.1 (Pin_1), J4.6 (Pin_6)
- net VCC: now reaches J3.9 (Pin_9)
- net VCC: now also J1.2 (Pin_2), J2.2 (Pin_2), J4.2 (Pin_2)
- net SDA: now reaches J1.3 (Pin_3)
- net SCK: now reaches J1.4 (Pin_4)
- net SCK: now also J4.3 (Pin_3)
- net RX: now reaches J2.3 (Pin_3)
- net TX: now reaches J2.4 (Pin_4)
- net MISO: now reaches J4.1 (Pin_1)
- net MOSI: now reaches J4.4 (Pin_4)
- net RST_N: now reaches J4.5 (Pin_5)
Other:
- moved on the sheet: J2, J3, J4

Commit message: placed footprints and made edge cut
Parts:
- renumbered J3 to J2, J2 to J3
Changed lines of the file:
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@@
 		(in_pos_files yes)
 		(dnp no)
-		(property "Reference" "J3"
+		(property "Reference" "J2"
 			(at 150.495 54.61 0)
 			(show_name no)
@@
 			(project "MCU_datalogger"
 				(path "/755fa3e0-2b76-4b1a-a49f-069f1564984c/66566ee9-3c88-4dbe-a111-e762fb8cc7c9"
-					(reference "J3")
+					(reference "J2")
 					(unit 1)
 				)
@@
 		(in_pos_files yes)
 		(dnp no)
-		(property "Reference" "J2"
+		(property "Reference" "J3"
 			(at 109.855 54.61 0)
 			(show_name no)
@@
 			(project "MCU_datalogger"
 				(path "/755fa3e0-2b76-4b1a-a49f-069f1564984c/66566ee9-3c88-4dbe-a111-e762fb8cc7c9"
-					(reference "J2")
+					(reference "J3")
 					(unit 1)
 				)

Commit message: fixed scl and sck bug in schematic
Connections:
- net SCK: no longer J1.4 (Pin_4)
- new net SCL: J1.4 (Pin_4)
Changed lines of the file:
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@@
 		)
 	)
-	(hierarchical_label "SCK"
+	(hierarchical_label "SCL"
 		(shape passive)
 		(at 78.74 67.31 0)
