File: MCU_datalogger.kicad_sch (KiCad schematic)
At the start: 25 parts, among them U1 24LC1025, U2 24LC1025, U3 DS1337S_, U4 ATMEGA328P-AU, Y1 32.768 KHz, Y2 16 MHz

Commit message: setup 2 layer PCB
Connections:
- net LED1_OUT: now reaches D1.1 (K), R7.1
- net CLK_16M: now reaches C2.2, U4.7 (PB6), Y2.1
- net X1: now reaches U3.1 (X1), Y1.2
- net X2: now reaches U3.2 (X2), Y1.1
- net INTA_N: now reaches R4.2, U3.3 (~{INTA})
- net SQW: now reaches R6.2, U3.7 (SQW/~INT)
- net AREF: now reaches C4.2, U4.20 (AREF)
- net CLK_16M_RTN: now reaches C3.2, U4.8 (PB7), Y2.2
- net LED2_OUT: now reaches D2.1 (K), R5.2
